File: hardware/driver-board/display.sch (KiCad schematic (older format))
At the start: 6 parts, among them U7 ER-TFT040-2

Commit message: Update display connector footprint to hand solder
Parts:
- U7: footprint Connector_FFC-FPC:TE_5-1734839-0_1x60-1MP_P0.5mm_Horizontal -> Connector_FFC-FPC:TE_5-1734839-0_1x60-1MP_P0.5mm_Horizontal_HandSolder
Changed lines of the file:
@@
 F 0 "U7" H 6078 4201 50  0000 L CNN
 F 1 "ER-TFT040-2" H 6078 4110 50  0000 L CNN
-F 2 "Connector_FFC-FPC:TE_5-1734839-0_1x60-1MP_P0.5mm_Horizontal" H 5750 6100 50  0001 C CNN
+F 2 "Connector_FFC-FPC:TE_5-1734839-0_1x60-1MP_P0.5mm_Horizontal_HandSolder" H 5750 6100 50  0001 C CNN
 F 3 "" H 5750 6100 50  0001 C CNN
 	1    5850 4100

Commit message: Adapt new SPI signal names from OSHWA
Parts:
- U7: symbol driver-board:ER-TFT040-2 -> driver-board-rescue:ER-TFT040-2-driver-board-driver-board-rescue
Connections:
- net CLK_3V renamed SCK_3V
- net MISO_3V renamed SDI_3V
- net MOSI_3V renamed SDO_3V
Changed lines of the file:
@@
 $EndDescr
 $Comp
-L driver-board:ER-TFT040-2 U7
+L driver-board-rescue:ER-TFT040-2-driver-board-driver-board-rescue U7
 U 1 1 5F09E273
 P 5850 4100
+AR Path="/5F09E273" Ref="U7"  Part="1"
+AR Path="/5F096907/5F09E273" Ref="U7"  Part="1"
 F 0 "U7" H 6078 4201 50  0000 L CNN
 F 1 "ER-TFT040-2" H 6078 4110 50  0000 L CNN
@@
 CS2_3V
 Text GLabel 5600 6000 0    50   Input ~ 0
-CLK_3V
+SCK_3V
 Text GLabel 5600 6100 0    50   Input ~ 0
 DC_3V
 Text GLabel 5600 6200 0    50   Input ~ 0
-MOSI_3V
+SDO_3V
 Text GLabel 5600 6300 0    50   Output ~ 0
-MISO_3V
+SDI_3V
 $Comp
 L power:GND #PWR052

Commit message: Add missing JLCPCB part numbers
Parts:
- C14: JLCPCB (none) -> C15849
- C15, C16: JLCPCB (none) -> C14663
- R4: JLCPCB (none) -> C22775
- R5: JLCPCB (none) -> C23178
Changed lines of the file:
@@
 F 2 "Resistor_SMD:R_0603_1608Metric" V 5030 1100 50  0001 C CNN
 F 3 "~" H 5100 1100 50  0001 C CNN
+F 4 "C22775" H 5100 1100 50  0001 C CNN "JLCPCB"
 	1    5100 1100
 	0    1    1    0
@@
 F 2 "Resistor_SMD:R_0603_1608Metric" V 2780 3100 50  0001 C CNN
 F 3 "~" H 2850 3100 50  0001 C CNN
+F 4 "C23178" H 2850 3100 50  0001 C CNN "JLCPCB"
 	1    2850 3100
 	0    1    1    0
@@
 F 2 "Capacitor_SMD:C_0603_1608Metric" H 3088 2650 50  0001 C CNN
 F 3 "~" H 3050 2800 50  0001 C CNN
+F 4 "C15849" H 3050 2800 50  0001 C CNN "JLCPCB"
 	1    3050 2800
 	1    0    0    -1
@@
 F 2 "Capacitor_SMD:C_0603_1608Metric" H 2638 4150 50  0001 C CNN
 F 3 "~" H 2600 4300 50  0001 C CNN
+F 4 "C14663" H 2600 4300 50  0001 C CNN "JLCPCB"
 	1    2600 4300
 	1    0    0    -1
@@
 F 2 "Capacitor_SMD:C_0603_1608Metric" H 3288 4150 50  0001 C CNN
 F 3 "~" H 3250 4300 50  0001 C CNN
+F 4 "C14663" H 3250 4300 50  0001 C CNN "JLCPCB"
 	1    3250 4300
 	1    0    0    -1

Commit message: Rename JLCPCB to LCSC and update PCB
Parts:
- C14: JLCPCB C15849 -> (none); LCSC (none) -> C15849
- C15, C16: JLCPCB C14663 -> (none); LCSC (none) -> C14663
- R4: JLCPCB C22775 -> (none); LCSC (none) -> C22775
- R5: JLCPCB C23178 -> (none); LCSC (none) -> C23178
Changed lines of the file:
@@
 F 2 "Resistor_SMD:R_0603_1608Metric" V 5030 1100 50  0001 C CNN
 F 3 "~" H 5100 1100 50  0001 C CNN
-F 4 "C22775" H 5100 1100 50  0001 C CNN "JLCPCB"
+F 4 "C22775" H 5100 1100 50  0001 C CNN "LCSC"
 	1    5100 1100
 	0    1    1    0
@@
 F 2 "Resistor_SMD:R_0603_1608Metric" V 2780 3100 50  0001 C CNN
 F 3 "~" H 2850 3100 50  0001 C CNN
-F 4 "C23178" H 2850 3100 50  0001 C CNN "JLCPCB"
+F 4 "C23178" H 2850 3100 50  0001 C CNN "LCSC"
 	1    2850 3100
 	0    1    1    0
@@
 F 2 "Capacitor_SMD:C_0603_1608Metric" H 3088 2650 50  0001 C CNN
 F 3 "~" H 3050 2800 50  0001 C CNN
-F 4 "C15849" H 3050 2800 50  0001 C CNN "JLCPCB"
+F 4 "C15849" H 3050 2800 50  0001 C CNN "LCSC"
 	1    3050 2800
 	1    0    0    -1
@@
 F 2 "Capacitor_SMD:C_0603_1608Metric" H 2638 4150 50  0001 C CNN
 F 3 "~" H 2600 4300 50  0001 C CNN
-F 4 "C14663" H 2600 4300 50  0001 C CNN "JLCPCB"
+F 4 "C14663" H 2600 4300 50  0001 C CNN "LCSC"
 	1    2600 4300
 	1    0    0    -1
@@
 F 2 "Capacitor_SMD:C_0603_1608Metric" H 3288 4150 50  0001 C CNN
 F 3 "~" H 3250 4300 50  0001 C CNN
-F 4 "C14663" H 3250 4300 50  0001 C CNN "JLCPCB"
+F 4 "C14663" H 3250 4300 50  0001 C CNN "LCSC"
 	1    3250 4300
 	1    0    0    -1

Commit message: Add drop-in replacement for buffer IC
Parts:
- R5: LCSC C23178 -> C25819
Changed lines of the file:
@@
 F 2 "Resistor_SMD:R_0603_1608Metric" V 2780 3100 50  0001 C CNN
 F 3 "~" H 2850 3100 50  0001 C CNN
-F 4 "C23178" H 2850 3100 50  0001 C CNN "LCSC"
+F 4 "C25819 " H 2850 3100 50  0001 C CNN "LCSC"
 	1    2850 3100
 	0    1    1    0
