File: hardware/driver-board/ft81x.sch (KiCad schematic (older format))
At the start: 7 parts, among them U6 FT813, X1 YSX321SL

Commit message: Add drop-in replacement for buffer IC
Parts:
- R3: LCSC C23178 -> C25819
Changed lines of the file:
@@
 F 2 "Resistor_SMD:R_0603_1608Metric" V 3830 2900 50  0001 C CNN
 F 3 "~" H 3900 2900 50  0001 C CNN
-F 4 "C23178" H 3900 2900 50  0001 C CNN "LCSC"
+F 4 "C25819 " H 3900 2900 50  0001 C CNN "LCSC"
 	1    3900 2900
 	0    1    1    0
