File: hardware/kicad/level-shifter.sch (KiCad schematic (older format))
At the start: 3 parts, among them U1 TXS0108E

Commit message: Add digikey bom alternative
Parts:
- C1, C2: DigiKey (none) -> 311-1335-1-ND
- U1: DigiKey (none) -> TXS0108EPWR
Changed lines of the file:
@@
 F 3 "~" H 5750 5300 50  0001 C CNN
 F 4 "C14663" H 5750 5300 50  0001 C CNN "LCSC"
+F 5 "311-1335-1-ND" H 5750 5300 50  0001 C CNN "DigiKey"
 	1    5750 5300
 	1    0    0    -1
@@
 F 3 "~" H 6450 5300 50  0001 C CNN
 F 4 "C14663" H 6450 5300 50  0001 C CNN "LCSC"
+F 5 "311-1335-1-ND" H 6450 5300 50  0001 C CNN "DigiKey"
 	1    6450 5300
 	1    0    0    -1
@@
 F 3 "" H 6100 4150 50  0001 C CNN
 F 4 "C17206" H 6100 4150 50  0001 C CNN "LCSC"
+F 5 "TXS0108EPWR" H 6100 4150 50  0001 C CNN "DigiKey"
 	1    6100 4150
 	1    0    0    -1

Commit message: Clean up board and expose less debug signals
Connections:
- net IRQ: now reaches U1.18 (B2)
- net IRQ_3V: now reaches U1.3 (A2)
- no-connect marks 4 -> 2
Changed lines of the file:
@@
 $EndComp
 NoConn ~ 6500 3700
-NoConn ~ 6500 3900
-NoConn ~ 5700 3900
 NoConn ~ 5700 3700
+Wire Wire Line
+	6500 3900 6750 3900
+Text GLabel 6750 3900 2    50   Output ~ 0
+IRQ
+Wire Wire Line
+	5700 3900 5450 3900
+Text GLabel 5450 3900 0    50   Input ~ 0
+IRQ_3V
 $EndSCHEMATC

Commit message: Update BOM
Parts:
- C1, C2: Description (none) -> CAP CER 0.1UF 16V X7R 0603; DigiKey 311-1335-1-ND -> (none); Manufacturer (none) -> Yageo; Mfg Part # (none) -> CC0603KPX7R7BB104
- U1: Description (none) -> IC TRNSLTR BIDIRECTIONAL 20TSSOP; DigiKey TXS0108EPWR -> (none); Manufacturer (none) -> Texas Instruments; Mfg Part # (none) -> TXS0108EPWR
Changed lines of the file:
@@
 F 3 "~" H 5750 5300 50  0001 C CNN
 F 4 "C14663" H 5750 5300 50  0001 C CNN "LCSC"
-F 5 "311-1335-1-ND" H 5750 5300 50  0001 C CNN "DigiKey"
+F 5 "" H 5750 5300 50  0001 C CNN "DigiKey"
+F 6 "CC0603KPX7R7BB104" H 5750 5300 50  0001 C CNN "Mfg Part #"
+F 7 "CAP CER 0.1UF 16V X7R 0603" H 5750 5300 50  0001 C CNN "Description"
+F 8 "Yageo" H 5750 5300 50  0001 C CNN "Manufacturer"
 	1    5750 5300
 	1    0    0    -1
@@
 F 3 "~" H 6450 5300 50  0001 C CNN
 F 4 "C14663" H 6450 5300 50  0001 C CNN "LCSC"
-F 5 "311-1335-1-ND" H 6450 5300 50  0001 C CNN "DigiKey"
+F 5 "" H 6450 5300 50  0001 C CNN "DigiKey"
+F 6 "CC0603KPX7R7BB104" H 6450 5300 50  0001 C CNN "Mfg Part #"
+F 7 "CAP CER 0.1UF 16V X7R 0603" H 6450 5300 50  0001 C CNN "Description"
+F 8 "Yageo" H 6450 5300 50  0001 C CNN "Manufacturer"
 	1    6450 5300
 	1    0    0    -1
@@
 F 3 "" H 6100 4150 50  0001 C CNN
 F 4 "C17206" H 6100 4150 50  0001 C CNN "LCSC"
-F 5 "TXS0108EPWR" H 6100 4150 50  0001 C CNN "DigiKey"
+F 5 "" H 6100 4150 50  0001 C CNN "DigiKey"
+F 6 "TXS0108EPWR" H 6100 4150 50  0001 C CNN "Mfg Part #"
+F 7 "IC TRNSLTR BIDIRECTIONAL 20TSSOP" H 6100 4150 50  0001 C CNN "Description"
+F 8 "Texas Instruments" H 6100 4150 50  0001 C CNN "Manufacturer"
 	1    6100 4150
 	1    0    0    -1
