File: hardware/kicad/miso-buffer.sch (KiCad schematic (older format))
At the start: 2 parts, among them U5 NC7SZ125

Commit message: Add digikey bom alternative
Parts:
- C9: DigiKey (none) -> 311-1335-1-ND
- U5: DigiKey (none) -> NC7SZ125M5X
Changed lines of the file:
@@
 F 3 "" H 5900 3900 50  0001 C CNN
 F 4 "C7420" H 5900 3950 50  0001 C CNN "LCSC"
+F 5 "NC7SZ125M5X" H 5900 3950 50  0001 C CNN "DigiKey"
 	1    5900 3950
 	1    0    0    -1
@@
 F 3 "~" H 5900 4650 50  0001 C CNN
 F 4 "C14663" H 5900 4650 50  0001 C CNN "LCSC"
+F 5 "311-1335-1-ND" H 5900 4650 50  0001 C CNN "DigiKey"
 	1    5900 4650
 	1    0    0    -1

Commit message: Update BOM
Parts:
- C9: Description (none) -> CAP CER 0.1UF 16V X7R 0603; DigiKey 311-1335-1-ND -> (none); Manufacturer (none) -> Yageo; Mfg Part # (none) -> CC0603KPX7R7BB104
- U5: Description (none) -> IC BUF NON-INVERT 5.5V SOT23-5; DigiKey NC7SZ125M5X -> (none); Manufacturer (none) -> ON Semiconductor; Mfg Part # (none) -> NC7SZ125M5X
Changed lines of the file:
@@
 F 3 "" H 5900 3900 50  0001 C CNN
 F 4 "C7420" H 5900 3950 50  0001 C CNN "LCSC"
-F 5 "NC7SZ125M5X" H 5900 3950 50  0001 C CNN "DigiKey"
+F 5 "" H 5900 3950 50  0001 C CNN "DigiKey"
+F 6 "NC7SZ125M5X" H 5900 3950 50  0001 C CNN "Mfg Part #"
+F 7 "IC BUF NON-INVERT 5.5V SOT23-5" H 5900 3950 50  0001 C CNN "Description"
+F 8 "ON Semiconductor" H 5900 3950 50  0001 C CNN "Manufacturer"
 	1    5900 3950
 	1    0    0    -1
@@
 F 3 "~" H 5900 4650 50  0001 C CNN
 F 4 "C14663" H 5900 4650 50  0001 C CNN "LCSC"
-F 5 "311-1335-1-ND" H 5900 4650 50  0001 C CNN "DigiKey"
+F 5 "" H 5900 4650 50  0001 C CNN "DigiKey"
+F 6 "CC0603KPX7R7BB104" H 5900 4650 50  0001 C CNN "Mfg Part #"
+F 7 "CAP CER 0.1UF 16V X7R 0603" H 5900 4650 50  0001 C CNN "Description"
+F 8 "Yageo" H 5900 4650 50  0001 C CNN "Manufacturer"
 	1    5900 4650
 	1    0    0    -1
