File: hardware/kicad/power.sch (KiCad schematic (older format))
At the start: 12 parts, among them U2 ME6210A30M3G, U3 ME6210A33M3G, U4 TLV61046ADB

Commit message: Update inductor in schematics
Parts:
- L1: Description FIXED IND 10UH 3MA 2.55 OHM SMD -> FIXED IND 10UH 220MA 2.6 OHM SMD; LCSC C1035 -> (none); Manufacturer Abracon LLC -> Taiyo Yuden; Mfg Part # AIML-0603-100K-T -> BRL1608T100M
Changed lines of the file:
@@
 F 2 "Inductor_SMD:L_0603_1608Metric" H 5750 3700 50  0001 C CNN
 F 3 "~" H 5750 3700 50  0001 C CNN
-F 4 "C1035" H 5750 3700 50  0001 C CNN "LCSC"
+F 4 "" H 5750 3700 50  0001 C CNN "LCSC"
 F 5 "" H 5750 3700 50  0001 C CNN "DigiKey"
-F 6 "AIML-0603-100K-T" H 5750 3700 50  0001 C CNN "Mfg Part #"
-F 7 "FIXED IND 10UH 3MA 2.55 OHM SMD" H 5750 3700 50  0001 C CNN "Description"
-F 8 "Abracon LLC" H 5750 3700 50  0001 C CNN "Manufacturer"
+F 6 "BRL1608T100M" H 5750 3700 50  0001 C CNN "Mfg Part #"
+F 7 "FIXED IND 10UH 220MA 2.6 OHM SMD" H 5750 3700 50  0001 C CNN "Description"
+F 8 "Taiyo Yuden" H 5750 3700 50  0001 C CNN "Manufacturer"
 	1    5750 3700
 	0    -1   -1   0

Commit message: Update BOM
Parts:
- U2: Manufacturer Diodes Incorporated -> MICRONE(Nanjing Micro One Elec); Mfg Part # AP2125N-3.0TRG1 -> ME6210A30M3G
- U3: Manufacturer Diodes Incorporated -> MICRONE(Nanjing Micro One Elec); Mfg Part # AP2125N-3.3TRG1 -> ME6210A33M3G
Changed lines of the file:
@@
 F 4 "C236680" H 4150 2150 50  0001 C CNN "LCSC"
 F 5 "" H 4150 2150 50  0001 C CNN "DigiKey"
-F 6 "AP2125N-3.3TRG1" H 4150 2150 50  0001 C CNN "Mfg Part #"
+F 6 "ME6210A33M3G" H 4150 2150 50  0001 C CNN "Mfg Part #"
 F 7 "IC REG LINEAR 3.3V 300MA SOT23-3" H 4150 2150 50  0001 C CNN "Description"
-F 8 "Diodes Incorporated" H 4150 2150 50  0001 C CNN "Manufacturer"
+F 8 "MICRONE(Nanjing Micro One Elec)" H 4150 2150 50  0001 C CNN "Manufacturer"
 	1    4150 2150
 	1    0    0    -1
@@
 F 4 "C116985" H 7200 2100 50  0001 C CNN "LCSC"
 F 5 "" H 7200 2100 50  0001 C CNN "DigiKey"
-F 6 "AP2125N-3.0TRG1" H 7200 2100 50  0001 C CNN "Mfg Part #"
+F 6 "ME6210A30M3G" H 7200 2100 50  0001 C CNN "Mfg Part #"
 F 7 "IC REG LINEAR 3V 300MA SOT23-3" H 7200 2100 50  0001 C CNN "Description"
-F 8 "Diodes Incorporated" H 7200 2100 50  0001 C CNN "Manufacturer"
+F 8 "MICRONE(Nanjing Micro One Elec)" H 7200 2100 50  0001 C CNN "Manufacturer"
 	1    7200 2100
 	1    0    0    -1
