File: extras/hardware/kicad/ft81x.sch (KiCad schematic (older format))
At the start: 7 parts, among them U6 FT813, X1 YSX321SL

Commit message: Update board to aisler specs
Parts:
- X1: DigiKey (none) -> RH100-12.000-12-1010-EXT-TR
Changed lines of the file:
@@
 F 3 "" H 5000 4000 50  0001 C CNN
 F 4 "C9002" H 5050 4000 50  0001 C CNN "LCSC"
-F 5 "" H 5050 4000 50  0001 C CNN "DigiKey"
+F 5 "RH100-12.000-12-1010-EXT-TR" H 5050 4000 50  0001 C CNN "DigiKey"
 F 6 "RH100-12.000-12-1010-EXT-TR" H 5050 4000 50  0001 C CNN "Mfg Part #"
 F 7 "XTAL 12MHZ 12PF SMD" H 5050 4000 50  0001 C CNN "Description"
