File: extras/hardware/kicad/ft81x.sch (KiCad schematic (older format))
At the start: 7 parts, among them U6 FT813, X1 YSX321SL

Commit message: Update parts bom
Parts:
- X1: value YSX321SL -> 12 MHz
Changed lines of the file:
@@
 P 5050 4000
 F 0 "X1" H 5050 4365 50  0000 C CNN
-F 1 "YSX321SL" H 5050 4274 50  0000 C CNN
+F 1 "12 MHz" H 5050 4274 50  0000 C CNN
 F 2 "Crystal:Crystal_SMD_3225-4Pin_3.2x2.5mm" H 5000 4000 50  0001 C CNN
 F 3 "" H 5000 4000 50  0001 C CNN
