File: extras/hardware/kicad/power.sch (KiCad schematic (older format))
At the start: 12 parts, among them U2 ME6210A30M3G, U3 ME6210A33M3G, U4 TLV61046ADB

Commit message: Update board to aisler specs
Parts:
- U2: DigiKey (none) -> AP2125N-3.0TRG1
- U3: DigiKey (none) -> P2125N-3.3TRG1
Changed lines of the file:
@@
 F 3 "" H 4150 2150 50  0001 C CNN
 F 4 "C236680" H 4150 2150 50  0001 C CNN "LCSC"
-F 5 "" H 4150 2150 50  0001 C CNN "DigiKey"
+F 5 "P2125N-3.3TRG1" H 4150 2150 50  0001 C CNN "DigiKey"
 F 6 "ME6210A33M3G" H 4150 2150 50  0001 C CNN "Mfg Part #"
 F 7 "IC REG LINEAR 3.3V 300MA SOT23-3" H 4150 2150 50  0001 C CNN "Description"
@@
 F 3 "" H 7200 2100 50  0001 C CNN
 F 4 "C116985" H 7200 2100 50  0001 C CNN "LCSC"
-F 5 "" H 7200 2100 50  0001 C CNN "DigiKey"
+F 5 "AP2125N-3.0TRG1" H 7200 2100 50  0001 C CNN "DigiKey"
 F 6 "ME6210A30M3G" H 7200 2100 50  0001 C CNN "Mfg Part #"
 F 7 "IC REG LINEAR 3V 300MA SOT23-3" H 7200 2100 50  0001 C CNN "Description"
