File: extras/hardware/kicad/power.sch (KiCad schematic (older format))
At the start: 12 parts, among them U2 ME6210A30M3G, U3 ME6210A33M3G, U4 TLV61046ADB

Commit message: Update parts bom
Parts:
- U2: value ME6210A30M3G -> 3.0V; Manufacturer MICRONE(Nanjing Micro One Elec) -> Diodes Incorporated; Mfg Part # ME6210A30M3G -> AP2125N-3.0TRG1
- U3: value ME6210A33M3G -> 3.3V; Manufacturer MICRONE(Nanjing Micro One Elec) -> Diodes Incorporated; Mfg Part # ME6210A33M3G -> AP2125N-3.3TRG1
Changed lines of the file:
@@
 P 4150 2150
 F 0 "U3" H 4150 2565 50  0000 C CNN
-F 1 "ME6210A33M3G" H 4150 2474 50  0000 C CNN
+F 1 "3.3V" H 4150 2474 50  0000 C CNN
 F 2 "Package_TO_SOT_SMD:SOT-23" H 4150 1400 50  0001 C CNN
 F 3 "" H 4150 2150 50  0001 C CNN
 F 4 "C236680" H 4150 2150 50  0001 C CNN "LCSC"
 F 5 "" H 4150 2150 50  0001 C CNN "DigiKey"
-F 6 "ME6210A33M3G" H 4150 2150 50  0001 C CNN "Mfg Part #"
+F 6 "AP2125N-3.3TRG1" H 4150 2150 50  0001 C CNN "Mfg Part #"
 F 7 "IC REG LINEAR 3.3V 300MA SOT23-3" H 4150 2150 50  0001 C CNN "Description"
-F 8 "MICRONE(Nanjing Micro One Elec)" H 4150 2150 50  0001 C CNN "Manufacturer"
+F 8 "Diodes Incorporated" H 4150 2150 50  0001 C CNN "Manufacturer"
 	1    4150 2150
 	1    0    0    -1
@@
 P 7200 2100
 F 0 "U2" H 7200 2515 50  0000 C CNN
-F 1 "ME6210A30M3G" H 7200 2424 50  0000 C CNN
+F 1 "3.0V" H 7200 2424 50  0000 C CNN
 F 2 "Package_TO_SOT_SMD:SOT-23" H 7200 1350 50  0001 C CNN
 F 3 "" H 7200 2100 50  0001 C CNN
 F 4 "C116985" H 7200 2100 50  0001 C CNN "LCSC"
 F 5 "" H 7200 2100 50  0001 C CNN "DigiKey"
-F 6 "ME6210A30M3G" H 7200 2100 50  0001 C CNN "Mfg Part #"
+F 6 "AP2125N-3.0TRG1" H 7200 2100 50  0001 C CNN "Mfg Part #"
 F 7 "IC REG LINEAR 3V 300MA SOT23-3" H 7200 2100 50  0001 C CNN "Description"
-F 8 "MICRONE(Nanjing Micro One Elec)" H 7200 2100 50  0001 C CNN "Manufacturer"
+F 8 "Diodes Incorporated" H 7200 2100 50  0001 C CNN "Manufacturer"
 	1    7200 2100
 	1    0    0    -1
