File: extras/hardware/kicad/display.sch (KiCad schematic (older format))
At the start: 5 parts, among them U7 ER-TFT040-2

Commit message: Clean up kicad project
Parts:
- U7: footprint kicad:HRS_FH28-60S-0.5SH(05) -> driver-board:HRS_FH28-60S-0.5SH(05)
Changed lines of the file:
@@
 F 0 "U7" H 6078 4201 50  0000 L CNN
 F 1 "ER-TFT040-2" H 6078 4110 50  0000 L CNN
-F 2 "kicad:HRS_FH28-60S-0.5SH(05)" H 5750 6100 50  0001 C CNN
+F 2 "driver-board:HRS_FH28-60S-0.5SH(05)" H 5750 6100 50  0001 C CNN
 F 3 "" H 5750 6100 50  0001 C CNN
 F 4 "" H 5850 4100 50  0001 C CNN "DigiKey"
